File: Airbeamv0_01.brd (EAGLE design)
At the start: 91.4 x 75.1 mm, 68 parts

Commit message: final revision 1
Parts:
- removed U_FB1: MF-MSMF050-2 500mA, rcl:L1812
- added U_FUSE: 1.8A, SparkFun-PowerIC:PTC-1206-WIDE
Connections:
- net VUSB: now also U_FUSE.2; no longer U_FB1.1
- net XUSB: now also U_FUSE.1; no longer U_FB1.2
Changed lines of the file:
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@@
 <attribute name="PARTNO" value="DNP" x="9.5" y="5" size="1.778" layer="27" display="off"/>
-</element>
-<element name="U_FB1" library="rcl" package="L1812" value="MF-MSMF050-2 500mA" x="13" y="63.915" smashed="yes" rot="R180">
-<attribute name="NAME" x="16.175" y="63.28" size="1.27" layer="49" font="vector" ratio="12"/>
-<attribute name="VALUE" x="15.794" y="62.264" size="1.27" layer="27" rot="R180"/>
-<attribute name="PARTNO" value="MH2029-300Y" x="13" y="63.915" size="1.778" layer="27" rot="R180" display="off"/>
 </element>
 <element name="U_Z1" library="varistor" package="CT/CN0603" value="CG0603MLC-05E" x="18" y="59.5" rot="R90">
@@
 <element name="UR_C1" library="SparkFun-Passives" package="0805" value="10uF" x="-48" y="-173">
 <attribute name="PARTNO" value="C2012X5R1C106K085AC" x="-48" y="-173" size="1.778" layer="27" display="off"/>
+</element>
+<element name="U_FUSE" library="SparkFun-PowerIC" package="PTC-1206-WIDE" value="1.8A" x="-47" y="-177">
+<attribute name="PARTNO" value="0ZCJ0100FF2E
+" x="-47" y="-177" size="1.778" layer="27" display="off"/>
 </element>
 </elements>
@@
 </signal>
 <signal name="XUSB" class="3">
-<contactref element="U_FB1" pad="2"/>
 <contactref element="CON_USB" pad="T1"/>
-<wire x1="5.125" y1="61" x2="11.05" y2="63.915" width="0" layer="19" extent="1-1"/>
+<contactref element="U_FUSE" pad="1"/>
+<wire x1="5.125" y1="61" x2="-48.654" y2="-177" width="0" layer="19" extent="1-1"/>
 </signal>
 <signal name="D2/SDA">
@@
 <contactref element="U_MEGA32U-Q" pad="7"/>
 <contactref element="ATMEGA32U4-T" pad="7"/>
-<contactref element="U_FB1" pad="1"/>
 <contactref element="VR_U" pad="4"/>
 <contactref element="VR_D1" pad="P$1"/>
@@
 <contactref element="U_C2" pad="1"/>
 <contactref element="VR_MOS-P1" pad="1"/>
+<contactref element="U_FUSE" pad="2"/>
+<wire x1="-45.346" y1="-177" x2="-45.95" y2="-174.1" width="0" layer="19" extent="1-1"/>
 <wire x1="-35.85" y1="-108" x2="-45.95" y2="-174.1" width="0" layer="19" extent="1-1"/>
 <wire x1="-35.9" y1="-104" x2="-35.85" y2="-108" width="0" layer="19" extent="1-1"/>
@@
 <wire x1="71.265" y1="23.01" x2="-15.05" y2="-46.1999" width="0" layer="19" extent="1-1"/>
 <wire x1="73.79" y1="23.31" x2="71.265" y2="23.01" width="0" layer="19" extent="1-1"/>
-<wire x1="14.95" y1="63.915" x2="71.265" y2="23.01" width="0" layer="19" extent="1-1"/>
 </signal>
 <signal name="AGND">

Commit message: r1_1
Parts:
- removed LED_ON: LED, Airbeam:LED_550
- removed LED_R1: (no value), SparkFun-Passives:0603-RES
- added CON_ADDON: BERG_1X5, Airbeam:BERG-5X1_SIDE
- CON_FAN: device Airbeam:FAN -> Airbeam:MOLEX_2PIN_SIDE
Connections:
- removed net N$2: LED_ON.CATHODE, LED_R1.2
- net +3V3: now also CON_ADDON.P$3
- net +5V: now also CON_ADDON.P$4
- net A1: now also CON_ADDON.P$1
- net A2: now also CON_ADDON.P$2
- net GND: now also CON_ADDON.P$5, CON_FAN.P$1; no longer CON_FAN.GND
- net VFAN: now also CON_FAN.P$2; no longer CON_FAN.VCC
Changed lines of the file:
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@@
 <attribute name="PARTNO" value="RC0603JR-070RL" x="-35.5" y="-139.5" size="1.778" layer="27" display="off"/>
 </element>
-<element name="CON_FAN" library="Airbeam" package="FAN" value="FAN" x="-40.5" y="-140">
-<attribute name="PARTNO" value="F16FB-05LLC /E" x="-40.5" y="-140" size="1.778" layer="27" display="off"/>
+<element name="CON_FAN" library="Airbeam" package="MOLEX_2PIN_SIDE" value="FAN" x="-40.5" y="-140">
+<attribute name="PARTNO" value="22-05-7025" x="-40.5" y="-140" size="1.778" layer="27" display="off"/>
 </element>
-<element name="LED_R1" library="SparkFun-Passives" package="0603-RES" value="" x="-41.5" y="-157"/>
-<element name="LED_ON" library="Airbeam" package="LED_550" value="LED" x="-39.5" y="-149.5"/>
 <element name="LED_R2" library="SparkFun-Passives" package="0603-RES" value="" x="-41.5" y="-174"/>
-<element name="LED_BT" library="Airbeam" package="LED_550" value="LED" x="-39.5" y="-166.5"/>
+<element name="LED_BT" library="Airbeam" package="LED_550" value="LED" x="-39.5" y="-166.5">
+<attribute name="PARTNO" value="550-1107F
+" x="-39.5" y="-166.5" size="1.778" layer="27" display="off"/>
+</element>
 <element name="VR_MOS-P1" library="Airbeam" package="SOT23" value="MOSFET-P" x="-45" y="-173">
 <attribute name="PARTNO" value="IRLML2246TRPBF " x="-45" y="-173" size="1.778" layer="27" display="off"/>
@@
 </element>
 <element name="U_FUSE" library="SparkFun-PowerIC" package="PTC-1206-WIDE" value="1.8A" x="-47" y="-177">
-<attribute name="PARTNO" value="0ZCJ0100FF2E
-" x="-47" y="-177" size="1.778" layer="27" display="off"/>
+<attribute name="PARTNO" value="0ZCJ0100FF2E " x="-47" y="-177" size="1.778" layer="27" display="off"/>
+</element>
+<element name="CON_ADDON" library="Airbeam" package="BERG-5X1_SIDE" value="BERG_1X5" x="-41" y="-188">
+<attribute name="PARTNO" value="PPTC051LGBN-RC
+" x="-41" y="-188" size="1.778" layer="27" display="off"/>
 </element>
 </elements>
@@
 <contactref element="CON_DUST" pad="P$3"/>
 <contactref element="UC_R2" pad="2"/>
+<contactref element="CON_ADDON" pad="P$4"/>
+<wire x1="-34.65" y1="-96.5" x2="-38.46" y2="-188" width="0" layer="19" extent="1-1"/>
 <wire x1="-21.5" y1="-86" x2="-34.65" y2="-96.5" width="0" layer="19" extent="1-1"/>
 <wire x1="-3.9" y1="-39.5" x2="-21.5" y2="-86" width="0" layer="19" extent="1-1"/>
@@
 <contactref element="UC_C4" pad="1"/>
 <contactref element="UC_R4" pad="1"/>
-<contactref element="CON_FAN" pad="GND"/>
+<contactref element="CON_FAN" pad="P$1"/>
 <contactref element="UR_C1" pad="2"/>
 <contactref element="UBT" pad="P$2"/>
-<wire x1="-39" y1="-140" x2="-47.1" y2="-173" width="0" layer="19" extent="1-1"/>
-<wire x1="-36.35" y1="-131.5" x2="-39" y2="-140" width="0" layer="19" extent="1-1"/>
+<contactref element="CON_ADDON" pad="P$5"/>
+<wire x1="-47.1" y1="-173" x2="-35.92" y2="-188" width="0" layer="19" extent="1-1"/>
+<wire x1="-41.75" y1="-140" x2="-47.1" y2="-173" width="0" layer="19" extent="1-1"/>
+<wire x1="-36.35" y1="-131.5" x2="-41.75" y2="-140" width="0" layer="19" extent="1-1"/>
 <wire x1="-35.85" y1="-128" x2="-36.35" y2="-131.5" width="0" layer="19" extent="1-1"/>
 <wire x1="-35.85" y1="-124" x2="-35.85" y2="-128" width="0" layer="19" extent="1-1"/>
@@
 <contactref element="U_MEGA32U-Q" pad="38"/>
 <contactref element="ATMEGA32U4-T" pad="38"/>
-<wire x1="67.19" y1="16.71" x2="67.49" y2="19.235" width="0" layer="19" extent="1-1"/>
+<contactref element="CON_ADDON" pad="P$2"/>
+<wire x1="67.19" y1="16.71" x2="-43.54" y2="-188" width="0" layer="19" extent="1-1"/>
+<wire x1="67.49" y1="19.235" x2="67.19" y2="16.71" width="0" layer="19" extent="1-1"/>
 </signal>
 <signal name="A1">
 <contactref element="U_MEGA32U-Q" pad="37"/>
 <contactref element="ATMEGA32U4-T" pad="37"/>
-<wire x1="66.39" y1="16.71" x2="66.99" y2="19.235" width="0" layer="19" extent="1-1"/>
+<contactref element="CON_ADDON" pad="P$1"/>
+<wire x1="66.39" y1="16.71" x2="-46.08" y2="-188" width="0" layer="19" extent="1-1"/>
+<wire x1="66.99" y1="19.235" x2="66.39" y2="16.71" width="0" layer="19" extent="1-1"/>
 </signal>
 <signal name="A0">
@@
 <contactref element="VR_R4" pad="1"/>
 <contactref element="VR_MOS-N1" pad="2"/>
+<contactref element="CON_ADDON" pad="P$3"/>
+<wire x1="-36.35" y1="-139.5" x2="-41" y2="-188" width="0" layer="19" extent="1-1"/>
 <wire x1="-34.55" y1="-137.1" x2="-36.35" y2="-139.5" width="0" layer="19" extent="1-1"/>
 <wire x1="-3.9" y1="-47.5" x2="-34.55" y2="-137.1" width="0" layer="19" extent="1-1"/>
@@
 <contactref element="VR_MOS-N1" pad="3"/>
 <contactref element="VR_R4" pad="2"/>
-<contactref element="CON_FAN" pad="VCC"/>
-<wire x1="-34.65" y1="-139.5" x2="-42" y2="-140" width="0" layer="19" extent="1-1"/>
+<contactref element="CON_FAN" pad="P$2"/>
+<wire x1="-34.65" y1="-139.5" x2="-39.25" y2="-140" width="0" layer="19" extent="1-1"/>
 <wire x1="-35.5" y1="-134.9" x2="-34.65" y2="-139.5" width="0" layer="19" extent="1-1"/>
 </signal>
-<signal name="N$2">
-<contactref element="LED_R1" pad="2"/>
-<contactref element="LED_ON" pad="CATHODE"/>
-<wire x1="-40.77" y1="-149.5" x2="-40.65" y2="-157" width="0" layer="19" extent="1-1"/>
-</signal>
 <signal name="N$3">

Commit message: got most parts placed, r2
Parts:
- removed U$2: (no value), Airbeam:SENSOR_DUST
- removed U_MOS: PUSHBUTTON, Airbeam:PUSHBUTTON
- added U$1, U$3: V_BUFFER, Airbeam:SOT23-5
- added U_ONOFF: PUSHBUTTON, Airbeam:PUSHBUTTON
- added VR3_0R1, VR5_0R2: 0, SparkFun-Passives:0603-RES
- added VR3_0R2, VR5_0R1: DNP, SparkFun-Passives:0603-RES
- CON_DUST: device Airbeam:RHT03 -> Airbeam:S4B-EH
- VDETECT: value VDETECT-RT9819 -> VDETEC_APX
- VR_MOS-N1: value MOSFET -> DNP
- VR_R3: value 0 -> DNP
- moved LED_BT 259.5 mm to (65.4, 70.8)
- moved VR_MOS-P1 234.0 mm to (15.5, 53.0), turned to 270 degrees
- moved U_FUSE 232.6 mm to (10.0, 48.5)
- moved VR_MOS-N1 221.5 mm to (38.0, 73.0), turned to 180 degrees
- moved VR_R4 218.8 mm to (34.0, 68.0)
- moved UR_C1 212.9 mm to (29.0, 25.5)
- moved CON_ADDON 209.2 mm to (2.86, 16.5), turned to 90 degrees
- moved U_C2 197.5 mm to (35.5, 76.5)
- moved U_C1 195.6 mm to (35.5, 78.5)
- moved CON_FAN 164.3 mm to (32.5, 7.24)
- moved LED_CH 144.4 mm to (7.62, 55.2), turned to 90 degrees
- moved VR_R2 142.0 mm to (27.0, 56.0)
- moved VR_R3 139.2 mm to (19.5, 53.0), turned to 90 degrees
- moved VR_D1 138.9 mm to (25.5, 68.5)
- moved UR_R1 137.3 mm to (25.0, 78.0)
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Connections:
- net A0 renamed A0/DUST_DETECT
- net IO9* renamed IO9*/TH_DETECT
- removed net D5*: ATMEGA32U4-T.31, U_MEGA32U-Q.31
- removed net IO13*: ATMEGA32U4-T.32, U_MEGA32U-Q.32
- removed net N$17: U_MOS.P$2, U_MOS.P$5, VDETECT.3, VR_R2.1
- removed net UC_FAN: VR_MOS-N1.1
- new net BT_RX: U$3.4, UBT.P$20
- new net BT_TX: U$1.2, UBT.P$21
- new net D5*/FAN_CONTROL: ATMEGA32U4-T.31, U_MEGA32U-Q.31, VR_MOS-N1.1
- new net IO13*/BT_LED: ATMEGA32U4-T.32, LED_BT.ANODE, U_MEGA32U-Q.32
- new net VDETECT_VDD: U_ONOFF.P$2, U_ONOFF.P$5, VDETECT.3, VR_R2.1
- new net VR3_PS: U_VR3.P$7, VR3_0R1.2, VR3_0R2.2
- new net VR5_PS: U_VR5.P$7, VR5_0R1.2, VR5_0R2.2
- net +3V3: now also U$3.5
- net +5V: now also U$1.5
- net GND: now also LED_R2.1, U$1.1, U$1.3, U$3.1, U$3.3, VR3_0R1.1, VR5_0R1.1; no longer U_VR3.P$7, U_VR5.P$7
- net IO10*/BT_TX: now also U$1.4; no longer UBT.P$21
- net IO11*/BT_RX: now also U$3.2; no longer UBT.P$20
- net VREG_IN: now also U_ONOFF.P$1, U_ONOFF.P$3, U_ONOFF.P$4, U_ONOFF.P$6, VR3_0R2.1, VR5_0R2.1; no longer U_MOS.P$1, U_MOS.P$3, U_MOS.P$4, U_MOS.P$6
Routing:
- net VEN: track 0.00 -> 48.2 mm, vias 0 -> 2
- net VREG_IN: track 0.00 -> 41.8 mm
- net N$4: track 0.00 -> 13.4 mm, vias 0 -> 3
- net N$10: track 0.00 -> 12.9 mm, vias 0 -> 3
- net D+: track 0.00 -> 11.7 mm
- net D-: track 0.00 -> 11.6 mm
- net VUSB: track 0.00 -> 9.63 mm
- net VR3_PS: track 0.00 -> 9.30 mm
- net +5V: track 0.00 -> 8.85 mm
- net +3V3: track 0.00 -> 8.85 mm
- net V_BAT: track 0.00 -> 6.01 mm
- net XUSB: track 0.00 -> 4.05 mm
- net N$9: track 0.00 -> 3.11 mm
- net N$12: track 0.00 -> 3.11 mm
- net N$11: track 0.00 -> 3.11 mm
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- added copper zone on layer 1, net UGND
Other:
- outline, holes or cut-outs redrawn

Commit message: 50% of board layed out, changes made
Parts:
- removed BUT_UC_RESET: TS42, SmartPrj:TS42
- removed VR_MOS-N1: DNP, Airbeam:SOT23
- added FAN_MOS-N1: DNP, Airbeam:SOT23
- added RESET_SWITCH: SWITCH, Airbeam:SWITCH_TACTILE
- moved LED_R2 264.5 mm to (60.5, 70.0), turned to 90 degrees
- moved UC_R4 190.3 mm to (66.0, 29.5), turned to 270 degrees
- moved UC_C6 178.0 mm to (58.5, 31.5)
- moved UC_C5 169.5 mm to (70.0, 17.0), turned to 270 degrees
- moved UC_C3 168.6 mm to (57.5, 13.0)
- moved UC_C4 167.6 mm to (61.5, 13.0), turned to 180 degrees
- moved UC_C7 159.5 mm to (50.0, 23.0), turned to 180 degrees
- moved UC_R1 144.2 mm to (59.5, 15.0), turned to 180 degrees
- moved UC_R3 142.5 mm to (10.0, 44.5), turned to 180 degrees
- moved UC_R2 138.1 mm to (48.0, 13.5), turned to 90 degrees
- moved VR_R4 64.5 mm to (34.0, 3.50), turned to 90 degrees
- moved UR_C1 47.5 mm to (29.0, 73.0), turned to 90 degrees
- moved CON_ICSP 37.1 mm to (42.9, 16.2)
- moved UC_CRYSTAL 34.1 mm to (59.5, 9.00), turned to 180 degrees
- moved UC_C2 29.4 mm to (52.0, 13.5), turned to 270 degrees
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Connections:
- removed net 5-GND: BUT_UC_RESET.5
- removed net N$5: UC_C1.1, UC_C2.1
- net +3V3: now also FAN_MOS-N1.2; no longer VR_MOS-N1.2
- net +5V: now also UC_C1.1, UC_C2.1
- net D5*/FAN_CONTROL: now also FAN_MOS-N1.1; no longer VR_MOS-N1.1
- net GND: now also RESET_SWITCH.P1, RESET_SWITCH.P2; no longer BUT_UC_RESET.3, BUT_UC_RESET.4
- net RESET: now also RESET_SWITCH.P3, RESET_SWITCH.P4; no longer BUT_UC_RESET.1, BUT_UC_RESET.2
- net VFAN: now also FAN_MOS-N1.3; no longer VR_MOS-N1.3
Routing:
- net IO13*/BT_LED: track 0.00 -> 58.5 mm, vias 0 -> 1
- net VEN: track 48.2 -> 3.92 mm
- net +5V: track 8.85 -> 53.0 mm, vias 0 -> 4
- net IO11*/BT_RX: track 0.00 -> 36.8 mm, vias 0 -> 2
- net RESET: track 0.00 -> 36.1 mm, vias 0 -> 1
- net VUSB: track 9.63 -> 32.7 mm
- net MOSI: track 0.00 -> 18.1 mm
- net MISO: track 0.00 -> 15.4 mm
- net SCK: track 0.00 -> 14.8 mm
- net XTAL1: track 0.00 -> 13.3 mm
- net XTAL2: track 0.00 -> 13.1 mm
- net GND: track 0.00 -> 13.1 mm, vias 1 -> 2
- net AVCC: track 0.00 -> 12.4 mm
- net BT_TX: track 0.00 -> 10.5 mm
- net UGND: track 2.77 -> 12.2 mm
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
Commit message: Updated BOM and schematic, still have to do personal full review. Having problems with eagle dru checking. Voltage regulator needs to be replaced
Parts:
- added U_Z3, U_Z4: CG0603MLC-05E, varistor:CT/CN0603
- R_LED_BT: value (none) -> 1.4k
- renumbered LED_R2 to R_LED_BT, UR_R1 to R_LED_CH
Changed lines of the file:
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@@
 <attribute name="PARTNO" value="MCP73831T-2ACI/OT" x="32.5" y="77" size="1.778" layer="27" rot="R270" display="off"/>
 </element>
-<element name="UR_R1" library="SparkFun-Passives" package="0603-RES" value="1.4k" x="24.5" y="77.5"/>
+<element name="R_LED_CH" library="SparkFun-Passives" package="0603-RES" value="1.4k" x="24.5" y="77.5">
+<attribute name="PARTNO" value="RC0603FR-071K4L" x="24.5" y="77.5" size="1.778" layer="27" display="off"/>
+</element>
 <element name="UR_R2" library="SparkFun-Passives" package="0603-RES" value="2K" x="25" y="74">
 <attribute name="PARTNO" value="RC0603FR-072KL" x="25" y="74" size="1.778" layer="27" display="off"/>
@@
 <attribute name="PARTNO" value="RC0603JR-070RL" x="19.5" y="53.5" size="1.778" layer="27" rot="R90" display="off"/>
 </element>
-<element name="CON_DUST" library="Airbeam" package="S4B-EH" value="CON_DUST" x="75.02" y="6.7" locked="yes"/>
+<element name="CON_DUST" library="Airbeam" package="S4B-EH" value="CON_DUST" x="75.02" y="6.7" locked="yes">
+<attribute name="PARTNO" value="S4B-EH" x="75.02" y="6.7" size="1.778" layer="27" display="off"/>
+</element>
 <element name="LED_CH" library="Airbeam" package="LED_550" value="LED" x="7.62" y="55.245" rot="R90">
 <attribute name="PARTNO" value="550-1307F" x="7.62" y="55.245" size="1.778" layer="27" rot="R90" display="off"/>
@@
 </element>
 <element name="UC_C5" library="SparkFun-Passives" package="0603-CAP" value="1uF" x="70" y="17" rot="R270">
-<attribute name="PARTNO" value="C2012X5R1C106K085AC" x="70" y="17" size="1.778" layer="27" rot="R270" display="off"/>
+<attribute name="PARTNO" value="C1608X5R1C105K080AA" x="70" y="17" size="1.778" layer="27" rot="R270" display="off"/>
 </element>
 <element name="UC_C6" library="SparkFun-Passives" package="0603-CAP" value="100nF" x="58.5" y="31.5">
-<attribute name="PARTNO" value="C2012X5R1C106K085AC" x="58.5" y="31.5" size="1.778" layer="27" display="off"/>
+<attribute name="PARTNO" value="C1608X7R1E104K080AA" x="58.5" y="31.5" size="1.778" layer="27" display="off"/>
 </element>
 <element name="UC_C4" library="SparkFun-Passives" package="0603-CAP" value="20pF" x="61.5" y="13" rot="R180">
@@
 <attribute name="PARTNO" value="22-05-7025" x="32.49995" y="7.235" size="1.778" layer="27" display="off"/>
 </element>
-<element name="LED_R2" library="SparkFun-Passives" package="0603-RES" value="" x="60.5" y="70" rot="R90"/>
+<element name="R_LED_BT" library="SparkFun-Passives" package="0603-RES" value="1.4k" x="60.5" y="70" rot="R90">
+<attribute name="PARTNO" value="RC0603FR-071K4L" x="60.5" y="70" size="1.778" layer="27" rot="R90" display="off"/>
+</element>
 <element name="LED_BT" library="Airbeam" package="LED_550" value="LED" x="65.405" y="70.8025">
 <attribute name="PARTNO" value="550-1107F " x="65.405" y="70.8025" size="1.778" layer="27" display="off"/>
@@
 <attribute name="PARTNO" value="RC0603JR-070RL" x="31" y="19.5" size="1.778" layer="27" display="off"/>
 </element>
-<element name="RESET_SWITCH" library="Airbeam" package="SWITCH_TACTILE" value="SWITCH" x="45.5" y="7.5" rot="R180"/>
+<element name="RESET_SWITCH" library="Airbeam" package="SWITCH_TACTILE" value="SWITCH" x="45.5" y="7.5" rot="R180">
+<attribute name="PARTNO" value="TL3315NF250Q" x="45.5" y="7.5" size="1.778" layer="27" rot="R180" display="off"/>
+</element>
+<element name="U_Z3" library="varistor" package="CT/CN0603" value="CG0603MLC-05E" x="-3.5" y="-3.5">
+<attribute name="PARTNO" value="CG0603MLC-05E" x="-3.5" y="-3.5" size="1.778" layer="27" font="vector" display="off"/>
+</element>
+<element name="U_Z4" library="varistor" package="CT/CN0603" value="CG0603MLC-05E" x="-3.5" y="-8.5">
+<attribute name="PARTNO" value="CG0603MLC-05E" x="-3.5" y="-8.5" size="1.778" layer="27" font="vector" display="off"/>
+</element>
 </elements>
 <signals>
@@
 <contactref element="UBT" pad="P$2"/>
 <contactref element="CON_ADDON" pad="P$5"/>
-<contactref element="LED_R2" pad="1"/>
+<contactref element="R_LED_BT" pad="1"/>
 <contactref element="U$3" pad="3"/>
 <contactref element="U$3" pad="1"/>
@@
 </signal>
 <signal name="N$14">
-<contactref element="UR_R1" pad="2"/>
+<contactref element="R_LED_CH" pad="2"/>
 <contactref element="LED_CH" pad="CATHODE"/>
 <wire x1="7.62" y1="53.975" x2="25.35" y2="77.5" width="0" layer="19" extent="1-1"/>
 </signal>
 <signal name="N$13">
-<contactref element="UR_R1" pad="1"/>
+<contactref element="R_LED_CH" pad="1"/>
 <contactref element="VR_U" pad="1"/>
 <wire x1="23.65" y1="77.5" x2="31.1999" y2="77.95" width="0" layer="19" extent="1-1"/>
@@
 </signal>
 <signal name="N$3">
-<contactref element="LED_R2" pad="2"/>
+<contactref element="R_LED_BT" pad="2"/>
 <contactref element="LED_BT" pad="CATHODE"/>
 <wire x1="64.135" y1="70.8025" x2="60.5475" y2="70.8025" width="0.2" layer="1"/>

Commit message: Board is nearing completion
Parts:
- removed VR_U: VREG-MCP73831, Airbeam:SOT23-5
- added U$2: VREG_MC34673, Airbeam:UFDFN-8
- added UC_C8: 1uF, SparkFun-Passives:0603-CAP
- added U_FB1: MH2029-300Y, wuerth-elektronik:0805
- added U_Z5, U_Z6: CG0603MLC-05E, varistor:CT/CN0603
- CON_ADDON: value BERG_1X5 -> CON_1X52MM; device Airbeam:BERG-5X1_SIDE -> Airbeam:CON_5_2MM
- UC_CRYSTAL: value (none) -> 16MHz
- UR_R2: value 2K -> 6.65k
- moved UC_R3 40.9 mm to (47.0, 27.0), turned to 90 degrees
- moved U_C1 32.1 mm to (23.3, 49.2), turned to 270 degrees
- moved U_C2 29.5 mm to (21.3, 49.2), turned to 270 degrees
- moved UR_R2 29.2 mm to (31.5, 45.5), turned to 90 degrees
- moved VR_R2 26.1 mm to (29.5, 30.0), turned to 180 degrees
- moved U_Z4 24.9 mm to (6.00, 14.5)
- moved UR_C1 24.3 mm to (33.0, 49.0), turned to 270 degrees
- moved R_LED_CH 23.3 mm to (12.5, 57.5), turned to 90 degrees
- moved VR5_C3 21.6 mm to (19.0, 3.50), turned to 180 degrees
- moved VR5_R1 20.6 mm to (29.5, 4.00), turned to 90 degrees
- moved U_R1 19.2 mm to (32.0, 40.5), turned to 270 degrees
- moved VR5_C2 19.0 mm to (19.0, 6.00), turned to 180 degrees
- moved U_Z3 18.6 mm to (6.00, 12.5)
- moved U_R2 18.2 mm to (32.0, 36.5), turned to 270 degrees
- moved VR5_L1 18.0 mm to (23.5, 3.50), turned to 0 degrees
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Connections:
- removed net AGND: ATMEGA32U4-T.43
- removed net N$15: UR_R2.1, VR_U.2
- new net N$7: CON_ADDON.P$5, U_FB1.1
- net +3V3: now also U_Z5.1
- net +5V: now also UC_C8.1, U_Z6.1
- net A1: now also U_Z3.1
- net A2: now also U_Z4.1
- net GND: now also ATMEGA32U4-T.43, CON_BAT.NC1, CON_BAT.NC2, U$2.P$4, U$2.P$5, U$2.P$9, UC_C8.2, UR_R2.1, U_FB1.2, U_Z3.2, U_Z4.2, U_Z5.2, U_Z6.2; no longer CON_ADDON.P$5
- net N$13: now also U$2.P$3; no longer VR_U.1
- net N$16: now also U$2.P$7; no longer VR_U.5
- net VUSB: now also U$2.P$1; no longer VR_U.4
- net V_BAT: now also U$2.P$8; no longer VR_U.3
Routing:
- net +5V: track 53.0 -> 160.2 mm, vias 4 -> 6
- net +3V3: track 11.0 -> 117.3 mm, vias 0 -> 7
- net A1: track 2.77 -> 91.5 mm, vias 0 -> 1
- net A2: track 2.65 -> 87.3 mm, vias 0 -> 1
- net D5*/FAN_CONTROL: track 2.91 -> 78.5 mm, vias 0 -> 4
- net VUSB: track 32.7 -> 107.8 mm, vias 0 -> 4
- net IO9*/TH_DETECT: track 2.66 -> 69.0 mm, vias 0 -> 3
- net UGND: track 12.2 -> 69.8 mm, vias 0 -> 2
- net A0/DUST_DETECT: track 2.90 -> 50.1 mm, vias 0 -> 1
- net VDETECT_VDD: track 0.00 -> 45.2 mm, vias 0 -> 1
- net VREG_IN: track 41.8 -> 82.0 mm, vias 0 -> 4
- net V_BAT: track 6.01 -> 44.8 mm, vias 0 -> 3
- net IO10*/BT_TX: track 2.78 -> 38.5 mm, vias 0 -> 4
- net RD-: track 7.00 -> 37.0 mm, vias 0 -> 2
- net VEN: track 3.92 -> 30.2 mm, vias 2 -> 3
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- added copper zone on layer 1, net +3V3
- added copper zone on layer 16, net +3V3
- added copper zone on layer 1, net +5V
- added copper zone on layer 16, net +5V
- added copper zone on layer 1, net GND
- added copper zone on layer 16, net GND
- added copper zone on layer 16, net VREG_IN
Other:
- outline, holes or cut-outs redrawn

Commit message: BOM exported and schematic checked again. Going to go through it and add prices
Parts:
- U_FB1, U_FB2: value MH2029-300Y -> (none)
Changed lines of the file:
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@@
 <attribute name="PARTNO" value="CG0603MLC-05E" x="30" y="40.5" size="1.778" layer="27" rot="R270" display="off"/>
 </element>
-<element name="U_FB2" library="wuerth-elektronik" package="0805" value="MH2029-300Y" x="15" y="39" rot="R270">
+<element name="U_FB2" library="wuerth-elektronik" package="0805" value="" x="15" y="39" rot="R270">
 <attribute name="PARTNO" value="MH2029-300Y" x="15" y="39" size="1.778" layer="27" rot="R270" display="off"/>
 </element>
@@
 <attribute name="PARTNO" value="CG0603MLC-05E" x="9.5" y="17.5" size="1.778" layer="27" rot="R270" display="off"/>
 </element>
-<element name="U_FB1" library="wuerth-elektronik" package="0805" value="MH2029-300Y" x="6.5" y="20.5">
+<element name="U_FB1" library="wuerth-elektronik" package="0805" value="" x="6.5" y="20.5">
 <attribute name="PARTNO" value="MH2029-300Y" x="6.5" y="20.5" size="1.778" layer="27" display="off"/>
 </element>
