File: Airbeamv0_01.brd (EAGLE design)
At the start: 91.4 x 75.1 mm, 78 parts

Commit message: updated prices. All parts (without Dust Sensor) = 0. Also added off-board parts to schematic
Parts:
- added 3_3V_FAN_COPOL, DUST_SENSOR, LION_BATTERY: OFF_BOARD, Airbeam:EMPTY
Changed lines of the file:
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@@
 <element name="CON_BAT" library="SparkFun-Connectors" package="JST-2-SMD" value="" x="22" y="34" locked="yes">
 <attribute name="PROD_ID" value="CONN-08352" x="22" y="34" size="1.778" layer="27" font="vector" display="off"/>
-<attribute name="PARTNO" value="CONN-08352" x="22" y="34" size="1.778" layer="27" display="off"/>
+<attribute name="PARTNO" value="S2B-PH-SM4-TB(LF)(SN)" x="22" y="34" size="1.778" layer="27" display="off"/>
 </element>
 <element name="R_LED_CH" library="SparkFun-Passives" package="0603-RES" value="1.4k" x="12.5" y="57.5" rot="R90">
@@
 <attribute name="PARTNO" value="MH2029-300Y" x="6.5" y="20.5" size="1.778" layer="27" display="off"/>
 </element>
+<element name="DUST_SENSOR" library="Airbeam" package="EMPTY" value="OFF_BOARD" x="-1" y="-1.5">
+<attribute name="PARTNO" value="PPD60PV-T2" x="-1" y="-1.5" size="1.778" layer="27" display="off"/>
+</element>
+<element name="3_3V_FAN_COPOL" library="Airbeam" package="EMPTY" value="OFF_BOARD" x="-2" y="-3">
+<attribute name="PARTNO" value="F16FB-05LLC/E" x="-2" y="-3" size="1.778" layer="27" display="off"/>
+</element>
+<element name="LION_BATTERY" library="Airbeam" package="EMPTY" value="OFF_BOARD" x="-3" y="-4.5">
+<attribute name="PARTNO" value="585460_2000mAh" x="-3" y="-4.5" size="1.778" layer="27" display="off"/>
+</element>
 </elements>
