File: Airbeamv0_01.sch (EAGLE design)
At the start: 77 parts

Commit message: BOM exported and schematic checked again. Going to go through it and add prices
Parts:
- U_FB1, U_FB2: value MH2029-300Y -> (none)
Changed lines of the file:
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@@
 <attribute name="PARTNO" value="CG0603MLC-05E"/>
 </part>
-<part name="U_FB2" library="wuerth-elektronik" deviceset="WE-CBF" device="_0805" value="MH2029-300Y">
+<part name="U_FB2" library="wuerth-elektronik" deviceset="WE-CBF" device="_0805">
 <attribute name="PARTNO" value="MH2029-300Y"/>
 </part>
@@
 <attribute name="PARTNO" value="CG0603MLC-05E"/>
 </part>
-<part name="U_FB1" library="wuerth-elektronik" deviceset="WE-CBF" device="_0805" value="MH2029-300Y">
+<part name="U_FB1" library="wuerth-elektronik" deviceset="WE-CBF" device="_0805">
 <attribute name="PARTNO" value="MH2029-300Y"/>
 </part>

Commit message: updated prices. All parts (without Dust Sensor) = 0. Also added off-board parts to schematic
Parts:
- added 3_3V_FAN_COPOL, DUST_SENSOR, LION_BATTERY: OFF_BOARD, Airbeam:PART_OFFBOARD
- CON_BAT: PARTNO CONN-08352 -> S2B-PH-SM4-TB(LF)(SN)
Other:
- note added: "OFF BOARD PARTS"
Changed lines of the file:
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@@
 <part name="GND25" library="supply1" deviceset="GND" device=""/>
 <part name="CON_BAT" library="SparkFun-Connectors" deviceset="JST_2MM_MALE" device="">
-<attribute name="PARTNO" value="CONN-08352"/>
+<attribute name="PARTNO" value="S2B-PH-SM4-TB(LF)(SN)"/>
 </part>
 <part name="GND26" library="supply1" deviceset="GND" device=""/>
@@
 </part>
 <part name="GND5" library="supply1" deviceset="GND" device=""/>
+<part name="DUST_SENSOR" library="Airbeam" deviceset="PART_OFFBOARD" device="" value="OFF_BOARD">
+<attribute name="PARTNO" value="PPD60PV-T2"/>
+</part>
+<part name="3_3V_FAN_COPOL" library="Airbeam" deviceset="PART_OFFBOARD" device="" value="OFF_BOARD">
+<attribute name="PARTNO" value="F16FB-05LLC/E"/>
+</part>
+<part name="LION_BATTERY" library="Airbeam" deviceset="PART_OFFBOARD" device="" value="OFF_BOARD">
+<attribute name="PARTNO" value="585460_2000mAh"/>
+</part>
 </parts>
 <sheets>
@@
 <wire x1="193.04" y1="-185.42" x2="193.04" y2="-170.18" width="0.1524" layer="97"/>
 <wire x1="193.04" y1="-170.18" x2="124.46" y2="-170.18" width="0.1524" layer="97"/>
+<text x="228.6" y="0" size="3.81" layer="94" ratio="10" rot="MR180" align="top-left">OFF BOARD PARTS</text>
 </plain>
 <instances>
@@
 </instance>
 <instance part="GND5" gate="1" x="-175.26" y="-193.04" rot="R270"/>
+<instance part="DUST_SENSOR" gate="G$1" x="238.76" y="-5.08">
+<attribute name="PARTNO" x="238.76" y="-5.08" size="1.778" layer="96" display="off"/>
+</instance>
+<instance part="3_3V_FAN_COPOL" gate="G$1" x="238.76" y="-15.24">
+<attribute name="PARTNO" x="238.76" y="-15.24" size="1.778" layer="96" display="off"/>
+</instance>
+<instance part="LION_BATTERY" gate="G$1" x="238.76" y="-25.4">
+<attribute name="PARTNO" x="238.76" y="-25.4" size="1.778" layer="96" display="off"/>
+</instance>
 </instances>
 <busses>

Commit message: Added library, updated board and schematic to reduce signal keepout
Parts:
- added BT_C1: 1uF, SparkFun-Passives:CAP0603-CAP
- CON_BAT: value (none) -> CON_BAT
- U_FB1: value (none) -> U_FB1
- U_FB2: value (none) -> U_FB2
- renumbered U$1 to U_BT_TX, U$3 to U_BT_RX
Connections:
- net +3V3: now also BT_C1.1
- net GND: now also BT_C1.2
Changed lines of the file:
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@@
 </variantdefs>
 <classes>
-<class number="0" name="default" width="0.254" drill="0.6096">
-<clearance class="0" value="0.254"/>
+<class number="0" name="default" width="0.1524" drill="0.3302">
+<clearance class="0" value="0.1524"/>
 </class>
-<class number="1" name="power" width="0.254" drill="0.6096">
-<clearance class="1" value="0.254"/>
+<class number="1" name="power" width="0.1524" drill="0.3302">
+<clearance class="1" value="0.1524"/>
 </class>
-<class number="2" name="gnd" width="0.254" drill="0.6096">
-<clearance class="2" value="0.254"/>
+<class number="2" name="gnd" width="0.1524" drill="0.3302">
+<clearance class="2" value="0.1524"/>
 </class>
-<class number="3" name="usbvcc" width="0.254" drill="0.6096">
-<clearance class="3" value="0.254"/>
+<class number="3" name="usbvcc" width="0.1524" drill="0.3302">
+<clearance class="3" value="0.1524"/>
 </class>
-<class number="4" name="aref" width="0.254" drill="0.6096">
-<clearance class="4" value="0.254"/>
+<class number="4" name="aref" width="0.1524" drill="0.3302">
+<clearance class="4" value="0.1524"/>
 </class>
 </classes>
@@
 <attribute name="PARTNO" value="CG0603MLC-05E"/>
 </part>
-<part name="U_FB2" library="wuerth-elektronik" deviceset="WE-CBF" device="_0805">
+<part name="U_FB2" library="wuerth-elektronik" deviceset="WE-CBF" device="_0805" value="U_FB2">
 <attribute name="PARTNO" value="MH2029-300Y"/>
 </part>
@@
 <part name="GND24" library="supply1" deviceset="GND" device=""/>
 <part name="GND25" library="supply1" deviceset="GND" device=""/>
-<part name="CON_BAT" library="SparkFun-Connectors" deviceset="JST_2MM_MALE" device="">
+<part name="CON_BAT" library="SparkFun-Connectors" deviceset="JST_2MM_MALE" device="" value="CON_BAT">
 <attribute name="PARTNO" value="S2B-PH-SM4-TB(LF)(SN)"/>
 </part>
@@
 <part name="+3V5" library="supply1" deviceset="+3V3" device=""/>
 <part name="GND34" library="supply1" deviceset="GND" device=""/>
-<part name="U$1" library="Airbeam" deviceset="V_BUFFER" device=""/>
-<part name="U$3" library="Airbeam" deviceset="V_BUFFER" device=""/>
+<part name="U_BT_TX" library="Airbeam" deviceset="V_BUFFER" device=""/>
+<part name="U_BT_RX" library="Airbeam" deviceset="V_BUFFER" device=""/>
 <part name="+3V6" library="supply1" deviceset="+3V3" device=""/>
 <part name="GND35" library="supply1" deviceset="GND" device=""/>
@@
 <attribute name="PARTNO" value="CG0603MLC-05E"/>
 </part>
-<part name="U_FB1" library="wuerth-elektronik" deviceset="WE-CBF" device="_0805">
+<part name="U_FB1" library="wuerth-elektronik" deviceset="WE-CBF" device="_0805" value="U_FB1">
 <attribute name="PARTNO" value="MH2029-300Y"/>
 </part>
@@
 <attribute name="PARTNO" value="585460_2000mAh"/>
 </part>
+<part name="BT_C1" library="SparkFun-Passives" deviceset="CAP" device="0603-CAP" value="1uF">
+<attribute name="PARTNO" value="C1608X5R1C105K080AA"/>
+</part>
+<part name="GND33" library="supply1" deviceset="GND" device=""/>
 </parts>
 <sheets>
@@
 <text x="335.28" y="132.08" size="2.54" layer="94">ALT3</text>
 <text x="-104.14" y="-114.3" size="3.81" layer="94">SENSORS</text>
-<text x="-370.84" y="-20.32" size="7.62" layer="94">TODO:
-</text>
+<text x="-360.68" y="27.94" size="7.62" layer="94">TODO:</text>
 <text x="48.26" y="-60.96" size="3.81" layer="94" ratio="10" rot="MR180" align="top-left">BATTERY</text>
 <text x="-139.7" y="0" size="6.35" layer="94">POWER</text>
@@
 <instance part="GND1" gate="1" x="-35.56" y="162.56" rot="R90"/>
 <instance part="GND12" gate="1" x="-93.98" y="175.26"/>
-<instance part="FID1" gate="G$1" x="20.32" y="33.02">
-<attribute name="PARTNO" x="20.32" y="33.02" size="1.778" layer="96" display="off"/>
-</instance>
-<instance part="FID2" gate="G$1" x="27.94" y="33.02">
-<attribute name="PARTNO" x="27.94" y="33.02" size="1.778" layer="96" display="off"/>
-</instance>
-<instance part="FID3" gate="G$1" x="35.56" y="33.02">
-<attribute name="PARTNO" x="35.56" y="33.02" size="1.778" layer="96" display="off"/>
+<instance part="FID1" gate="G$1" x="238.76" y="-60.96">
+<attribute name="PARTNO" x="238.76" y="-60.96" size="1.778" layer="96" display="off"/>
+</instance>
+<instance part="FID2" gate="G$1" x="246.38" y="-60.96">
+<attribute name="PARTNO" x="246.38" y="-60.96" size="1.778" layer="96" display="off"/>
+</instance>
+<instance part="FID3" gate="G$1" x="254" y="-60.96">
+<attribute name="PARTNO" x="254" y="-60.96" size="1.778" layer="96" display="off"/>
 </instance>
 <instance part="U_Z1" gate="G$1" x="-96.52" y="-68.58" smashed="yes" rot="R90">
@@
 <instance part="+3V5" gate="G$1" x="-127" y="-198.12" rot="R180"/>
 <instance part="GND34" gate="1" x="76.2" y="-157.48"/>
-<instance part="U$1" gate="G$1" x="38.1" y="-147.32"/>
-<instance part="U$3" gate="G$1" x="38.1" y="-172.72" rot="R180"/>
+<instance part="U_BT_TX" gate="G$1" x="38.1" y="-147.32"/>
+<instance part="U_BT_RX" gate="G$1" x="38.1" y="-172.72" rot="R180"/>
 <instance part="+3V6" gate="G$1" x="43.18" y="-182.88" rot="R270"/>
 <instance part="GND35" gate="1" x="45.72" y="-165.1" rot="R90"/>
@@
 <attribute name="PARTNO" x="238.76" y="-25.4" size="1.778" layer="96" display="off"/>
 </instance>
+<instance part="BT_C1" gate="G$1" x="-35.56" y="-154.94">
+<attribute name="PARTNO" x="-35.56" y="-154.94" size="1.778" layer="96" display="off"/>
+</instance>
+<instance part="GND33" gate="1" x="-35.56" y="-165.1"/>
 </instances>
 <busses>
@@
 </segment>
 <segment>
-<pinref part="U$1" gate="G$1" pin="VCC"/>
+<pinref part="U_BT_TX" gate="G$1" pin="VCC"/>
 <wire x1="38.1" y1="-144.78" x2="38.1" y2="-139.7" width="0.1524" layer="91"/>
 <wire x1="38.1" y1="-139.7" x2="40.64" y2="-139.7" width="0.1524" layer="91"/>
@@
 </segment>
 <segment>
-<pinref part="U$3" gate="G$1" pin="GND"/>
+<pinref part="U_BT_RX" gate="G$1" pin="GND"/>
 <wire x1="38.1" y1="-170.18" x2="38.1" y2="-165.1" width="0.1524" layer="91"/>
 <wire x1="38.1" y1="-165.1" x2="40.64" y2="-165.1" width="0.1524" layer="91"/>
 <pinref part="GND35" gate="1" pin="GND"/>
-<pinref part="U$3" gate="G$1" pin="OE_N"/>
+<pinref part="U_BT_RX" gate="G$1" pin="OE_N"/>
 <wire x1="40.64" y1="-165.1" x2="43.18" y2="-165.1" width="0.1524" layer="91"/>
 <wire x1="40.64" y1="-170.18" x2="40.64" y2="-165.1" width="0.1524" layer="91"/>
@@
 </segment>
 <segment>
-<pinref part="U$1" gate="G$1" pin="GND"/>
+<pinref part="U_BT_TX" gate="G$1" pin="GND"/>
 <wire x1="38.1" y1="-149.86" x2="38.1" y2="-154.94" width="0.1524" layer="91"/>
 <wire x1="38.1" y1="-154.94" x2="40.64" y2="-154.94" width="0.1524" layer="91"/>
-<pinref part="U$1" gate="G$1" pin="OE_N"/>
+<pinref part="U_BT_TX" gate="G$1" pin="OE_N"/>
 <wire x1="35.56" y1="-149.86" x2="35.56" y2="-154.94" width="0.1524" layer="91"/>
 <wire x1="35.56" y1="-154.94" x2="38.1" y2="-154.94" width="0.1524" layer="91"/>
@@
 <wire x1="149.86" y1="86.36" x2="129.54" y2="86.36" width="0.1524" layer="91"/>
 <label x="142.24" y="86.36" size="1.778" layer="95"/>
+</segment>
+<segment>
+<pinref part="BT_C1" gate="G$1" pin="2"/>
+<wire x1="-35.56" y1="-157.48" x2="-35.56" y2="-162.56" width="0.1524" layer="91"/>
+<pinref part="GND33" gate="1" pin="GND"/>
 </segment>
 </net>
@@
 <pinref part="UBT" gate="G$1" pin="P$12"/>
 <wire x1="-38.1" y1="-144.78" x2="-38.1" y2="-147.32" width="0.1524" layer="91"/>
-<wire x1="-38.1" y1="-147.32" x2="-15.24" y2="-147.32" width="0.1524" layer="91"/>
+<wire x1="-38.1" y1="-147.32" x2="-35.56" y2="-147.32" width="0.1524" layer="91"/>
 <label x="-35.56" y="-147.32" size="1.778" layer="95"/>
+<pinref part="BT_C1" gate="G$1" pin="1"/>
+<wire x1="-35.56" y1="-147.32" x2="-15.24" y2="-147.32" width="0.1524" layer="91"/>
+<wire x1="-35.56" y1="-149.86" x2="-35.56" y2="-147.32" width="0.1524" layer="91"/>
+<junction x="-35.56" y="-147.32"/>
 </segment>
 <segment>
@@
 </segment>
 <segment>
-<pinref part="U$3" gate="G$1" pin="VCC"/>
+<pinref part="U_BT_RX" gate="G$1" pin="VCC"/>
 <wire x1="38.1" y1="-175.26" x2="38.1" y2="-182.88" width="0.1524" layer="91"/>
 <wire x1="38.1" y1="-182.88" x2="40.64" y2="-182.88" width="0.1524" layer="91"/>
@@
 </segment>
 <segment>
-<pinref part="U$3" gate="G$1" pin="A"/>
+<pinref part="U_BT_RX" gate="G$1" pin="A"/>
 <wire x1="40.64" y1="-172.72" x2="53.34" y2="-172.72" width="0.1524" layer="91"/>
 <label x="48.26" y="-172.72" size="1.778" layer="95"/>
@@
 </segment>
 <segment>
-<pinref part="U$1" gate="G$1" pin="Y"/>
+<pinref part="U_BT_TX" gate="G$1" pin="Y"/>
 <wire x1="40.64" y1="-147.32" x2="53.34" y2="-147.32" width="0.1524" layer="91"/>
 <label x="48.26" y="-147.32" size="1.778" layer="95"/>
@@
 <segment>
 <pinref part="VR3_0R2" gate="G$1" pin="1"/>
-<wire x1="152.4" y1="-60.96" x2="152.4" y2="-63.5" width="0.1524" layer="91"/>
-<label x="154.94" y="-83.82" size="1.778" layer="95" rot="R90"/>
+<wire x1="152.4" y1="-60.96" x2="152.4" y2="-66.04" width="0.1524" layer="91"/>
+<label x="154.94" y="-73.66" size="1.778" layer="95" rot="R90"/>
 </segment>
 <segment>
 <pinref part="VR5_0R2" gate="G$1" pin="1"/>
-<wire x1="149.86" y1="-127" x2="149.86" y2="-132.08" width="0.1524" layer="91"/>
+<wire x1="149.86" y1="-127" x2="149.86" y2="-134.62" width="0.1524" layer="91"/>
 <label x="152.4" y="-137.16" size="1.778" layer="95" rot="R90"/>
 </segment>
@@
 <pinref part="UBT" gate="G$1" pin="P$21"/>
 <label x="17.78" y="-147.32" size="1.778" layer="95"/>
-<pinref part="U$1" gate="G$1" pin="A"/>
+<pinref part="U_BT_TX" gate="G$1" pin="A"/>
 <wire x1="2.54" y1="-147.32" x2="35.56" y2="-147.32" width="0.1524" layer="91"/>
 </segment>
@@
 <label x="17.78" y="-149.86" size="1.778" layer="95"/>
 <wire x1="27.94" y1="-149.86" x2="27.94" y2="-172.72" width="0.1524" layer="91"/>
-<pinref part="U$3" gate="G$1" pin="Y"/>
+<pinref part="U_BT_RX" gate="G$1" pin="Y"/>
 <wire x1="27.94" y1="-172.72" x2="35.56" y2="-172.72" width="0.1524" layer="91"/>
 </segment>
@@
 </sheet>
 </sheets>
+<errors>
+</errors>
 </schematic>
 </drawing>

Commit message: Added Airwires, ready for review
Parts:
- U_MEGA32U-Q: value ATMEGA32U4-XUMU -> DNP
Changed lines of the file:
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@@
 </part>
 <part name="GND3" library="supply1" deviceset="GND" device=""/>
-<part name="U_MEGA32U-Q" library="SmartPrj" deviceset="ATMEGA32U4-XU" device="MU">
+<part name="U_MEGA32U-Q" library="SmartPrj" deviceset="ATMEGA32U4-XU" device="MU" value="DNP">
 <attribute name="PARTNO" value="DNP"/>
 </part>

Commit message: Board updated, Gerber added, ready for review
Parts:
- added BT_C2, VR5_C4: 100nF, SparkFun-Passives:CAP0603-CAP
- added CD_C1, CE_C1, CTH_C1: 1uF, SparkFun-Passives:CAP0603-CAP
- renumbered U$2 to U_VRUSB
Connections:
- net +5V: now also BT_C2.1, CD_C1.1, CE_C1.1, CTH_C1.1
- net GND: now also BT_C2.2, CD_C1.2, CE_C1.2, CTH_C1.2, VR5_C4.2
- net VREG_IN: now also VR5_C4.1
